File: RiscPcPcbRepair/RiscPcPcbRepair.kicad_sch (KiCad schematic)
At the start: 21 parts, among them IC33 74ACT244

Commit message: Completeldy PCB
Parts:
- added +5V2, GND2, GND3, GND4: TestPoint_Small, TestPoint:TestPoint_THTPad_1.0x1.0mm_Drill0.5mm, symbol Connector:TestPoint_Small
- added C1, C2: 100n, Capacitor_SMD:C_0805_2012Metric, symbol Device:C
Connections:
- net +5V: now also C1.1
- net GND: now also C1.2, C2.1, GND2.1, GND3.1, GND4.1
- new net: +5V2.1, C2.2
