File: RiscPcRtcRepair/RiscPcRtcRepair.kicad_sch (KiCad schematic)
At the start: 0 parts

Commit message: Updte RTC schematic and notes
Parts:
- added BT1: CR2032, Battery:BatteryHolder_Keystone_3034_1x20mm, symbol Device:Battery
- added C1: 18pF, Capacitor_SMD:C_0402_1005Metric, symbol Device:C
- added C2: 15pF, Capacitor_SMD:C_0402_1005Metric, symbol Device:C
- added C3: 4.7uF, Capacitor_SMD:C_0402_1005Metric, symbol Device:C
- added D1: BAT85, Diode_SMD:D_SOD-323, symbol Device:D_Schottky
- added F1, GND1: TestPoint, TestPoint:TestPoint_THTPad_1.5x1.5mm_Drill0.7mm, symbol Connector:TestPoint
- added F2, SCL1, SDA1: TestPoint, symbol Connector:TestPoint
- added INT#1: TestPoint, TestPoint:TestPoint_Pad_2.0x2.0mm, symbol Connector:TestPoint
- added U1: PCF8583, Package_SO:SOIC-8_3.9x4.9mm_P1.27mm, symbol Local:PCF8583
- added X1: 32.768kHz, Crystal:Crystal_HC49-4H_Vertical, symbol Device:Crystal
Connections:
- new net: SDA1.1, U1.5 (SDA)
- new net: C1.2, C2.2, U1.1 (OSCI), X1.1
- new net: INT#1.1, U1.7 (~{INT})
- new net: U1.2 (OSCO), X1.2
- new net: BT1.1 (+), D1.2 (A)
- new net: SCL1.1, U1.6 (SCL)
- new net +5V: C1.1, C2.1, C3.1, D1.1 (K), U1.8 (VDD)
- new net GND: BT1.2 (-), C3.2, F1.1, F2.1, GND1.1, U1.3 (A0), U1.4 (VSS)

Commit message: Finished RTC repair board
Parts:
- removed F1: TestPoint, TestPoint:TestPoint_THTPad_1.5x1.5mm_Drill0.7mm, symbol Connector:TestPoint
- removed F2: TestPoint, symbol Connector:TestPoint
- added +5V1: TestPoint, symbol Connector:TestPoint
- added D1: BAT85, Diode_SMD:D_SOD-323, symbol Device:D_Schottky
- BT1: footprint Battery:BatteryHolder_Keystone_3034_1x20mm -> Battery:Battery_Panasonic_CR2032-HFN_Horizontal_CircularHoles
- C3: footprint Capacitor_SMD:C_0402_1005Metric -> Capacitor_SMD:C_Elec_4x5.4
- GND1: footprint TestPoint:TestPoint_THTPad_1.5x1.5mm_Drill0.7mm -> (none)
- SCL1, SDA1: footprint (none) -> TestPoint:TestPoint_THTPad_D1.5mm_Drill0.7mm
- X1: footprint Crystal:Crystal_HC49-4H_Vertical -> Crystal:Crystal_C38-LF_D3.0mm_L8.0mm_Horizontal_1EP_style2
- renumbered D1 to D2, INT#1 to INT1
Connections:
- net +5V: now also +5V1.1, D1.2 (A); no longer C1.1, C2.1, C3.1, D2.1 (K), U1.8 (VDD)
- new net: C1.1, C2.1, C3.1, D1.1 (K), D2.1 (K), U1.8 (VDD)
