File: RiscPcRtcRepair/RiscPcRtcRepair.kicad_sch (KiCad schematic)
At the start: 16 parts, among them U1 PCF8583T, Y1 Crystal_GND3

Commit message: Fix warnings and add gerbers
Parts:
- Y1: footprint Crystal:Crystal_C38-LF_D3.0mm_L8.0mm_Horizontal_1EP_style1 -> Crystal:Crystal_C26-LF_D2.1mm_L6.5mm_Horizontal_1EP_style2
- renumbered +5V2 to +5V1, +5V1 to +5V2, C4 to C3, C3 to C4
Changed lines of the file:
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@@
 		(dnp no)
 		(fields_autoplaced yes)
-		(property "Reference" "+5V1"
+		(property "Reference" "+5V2"
 			(at 147.32 71.6279 0)
 			(effects
@@
 			(project "RiscPcRtcRepair"
 				(path "/7dd0612d-24f5-436a-9fd4-f1ef6c878b14"
-					(reference "+5V1")
+					(reference "+5V2")
 					(unit 1)
 				)
@@
 		(dnp no)
 		(fields_autoplaced yes)
-		(property "Reference" "#PWR01"
+		(property "Reference" "#PWR02"
 			(at 100.33 134.62 0)
 			(effects
@@
 			(project "RiscPcRtcRepair"
 				(path "/7dd0612d-24f5-436a-9fd4-f1ef6c878b14"
-					(reference "#PWR01")
+					(reference "#PWR02")
 					(unit 1)
 				)
@@
 		(dnp no)
 		(fields_autoplaced yes)
-		(property "Reference" "C4"
+		(property "Reference" "C3"
 			(at 120.65 91.44 90)
 			(effects
@@
 			(project "RiscPcRtcRepair"
 				(path "/7dd0612d-24f5-436a-9fd4-f1ef6c878b14"
-					(reference "C4")
+					(reference "C3")
 					(unit 1)
 				)
@@
 			)
 		)
-		(property "Footprint" "Crystal:Crystal_C38-LF_D3.0mm_L8.0mm_Horizontal_1EP_style1"
+		(property "Footprint" "Crystal:Crystal_C26-LF_D2.1mm_L6.5mm_Horizontal_1EP_style2"
 			(at 92.71 111.76 0)
 			(effects
@@
 		(on_board yes)
 		(dnp no)
-		(property "Reference" "#PWR06"
+		(property "Reference" "#PWR01"
 			(at 92.71 123.19 0)
 			(effects
@@
 			(project "RiscPcRtcRepair"
 				(path "/7dd0612d-24f5-436a-9fd4-f1ef6c878b14"
-					(reference "#PWR06")
+					(reference "#PWR01")
 					(unit 1)
 				)
@@
 		(on_board yes)
 		(dnp no)
-		(property "Reference" "#PWR02"
+		(property "Reference" "#PWR04"
 			(at 121.92 77.216 0)
 			(effects
@@
 			(project "RiscPcRtcRepair"
 				(path "/7dd0612d-24f5-436a-9fd4-f1ef6c878b14"
-					(reference "#PWR02")
+					(reference "#PWR04")
 					(unit 1)
 				)
@@
 		(dnp no)
 		(fields_autoplaced yes)
-		(property "Reference" "#PWR04"
+		(property "Reference" "#PWR06"
 			(at 158.75 104.14 0)
 			(effects
@@
 			(project "RiscPcRtcRepair"
 				(path "/7dd0612d-24f5-436a-9fd4-f1ef6c878b14"
-					(reference "#PWR04")
+					(reference "#PWR06")
 					(unit 1)
 				)
@@
 		(on_board yes)
 		(dnp no)
-		(property "Reference" "C3"
+		(property "Reference" "C4"
 			(at 135.89 92.71 0)
 			(effects
@@
 			(project "RiscPcRtcRepair"
 				(path "/7dd0612d-24f5-436a-9fd4-f1ef6c878b14"
-					(reference "C3")
+					(reference "C4")
 					(unit 1)
 				)
@@
 		(dnp no)
 		(fields_autoplaced yes)
-		(property "Reference" "+5V2"
+		(property "Reference" "+5V1"
 			(at 137.16 71.6279 0)
 			(effects
@@
 			(project "RiscPcRtcRepair"
 				(path "/7dd0612d-24f5-436a-9fd4-f1ef6c878b14"
-					(reference "+5V2")
+					(reference "+5V1")
 					(unit 1)
 				)
@@
 		(on_board yes)
 		(dnp no)
-		(property "Reference" "#PWR03"
+		(property "Reference" "#PWR05"
 			(at 138.43 104.14 0)
 			(effects
@@
 			(project "RiscPcRtcRepair"
 				(path "/7dd0612d-24f5-436a-9fd4-f1ef6c878b14"
-					(reference "#PWR03")
+					(reference "#PWR05")
 					(unit 1)
 				)
@@
 		(dnp no)
 		(fields_autoplaced yes)
-		(property "Reference" "#PWR05"
+		(property "Reference" "#PWR03"
 			(at 110.49 99.06 0)
 			(effects
@@
 			(project "RiscPcRtcRepair"
 				(path "/7dd0612d-24f5-436a-9fd4-f1ef6c878b14"
-					(reference "#PWR05")
-					(unit 1)
-				)
+					(reference "#PWR03")
+					(unit 1)
+				)

Commit message: change diode to TS4148
Higher voltage drop but that doesn't matter but crucially Schottky
diodes are not suitable for this application as they have reverse current
leakage which whilst probably fine isn't ideal in this application.
Parts:
- D1, D2: value BAT46W -> TS4148
Changed lines of the file:
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@@
 			)
 		)
-		(property "Value" "BAT46W"
+		(property "Value" "TS4148"
 			(at 118.618 81.28 0)
 			(effects
@@
 			)
 		)
-		(property "Value" "BAT46W"
+		(property "Value" "TS4148"
 			(at 148.59 81.788 0)
 			(effects

Commit message: Update notes and add bench test scripts
Parts:
- C3: value C -> 100nF
- D1, D2: symbol Device:D_Schottky -> Device:D
Changed lines of the file:
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@@
 	)
 	(symbol
-		(lib_id "Device:D_Schottky")
+		(lib_id "Device:D")
 		(at 121.92 81.28 90)
 		(unit 1)
@@
 			)
 		)
-		(property "Description" "Schottky diode"
+		(property "Description" "Diode"
+			(at 121.92 81.28 0)
+			(effects
+				(font
+					(size 1.27 1.27)
+				)
+				(hide yes)
+			)
+		)
+		(property "Sim.Device" "D"
+			(at 121.92 81.28 0)
+			(effects
+				(font
+					(size 1.27 1.27)
+				)
+				(hide yes)
+			)
+		)
+		(property "Sim.Pins" "1=K 2=A"
 			(at 121.92 81.28 0)
 			(effects
@@
 			)
 		)
-		(property "Value" "C"
+		(property "Value" "100nF"
 			(at 120.65 93.98 90)
 			(effects
@@
 	)
 	(symbol
-		(lib_id "Device:D_Schottky")
+		(lib_id "Device:D")
 		(at 148.59 85.09 0)
 		(unit 1)
@@
 			)
 		)
-		(property "Description" "Schottky diode"
+		(property "Description" "Diode"
 			(at 148.59 85.09 0)
 			(effects
+				(font
+					(size 1.27 1.27)
+				)
+				(hide yes)
+			)
+		)
+		(property "Sim.Device" "D"
+			(at 148.59 85.09 0)
+			(effects
+				(font
+					(size 1.27 1.27)
+				)
+				(hide yes)
+			)
+		)
+		(property "Sim.Pins" "1=K 2=A"
+			(at 148.59 85.09 0)
+			(effects
